File: STM32H755_template/STM32H755_template.kicad_pcb (KiCad board)
At the start: 2 copper layers, 59 parts, among them IC1 LV14340DDAR, IC2 W25M512JVFIQ, J2 melex ultra fit, J3 melex ultra fit, J4 molex ultrafit, J5 molex ultrafit, J6 molex ultrafit, J7 molex ultrafit, J9 RJ45, K1 EC2-3NU, K2 EC2-3NU, SW1 RST_BTN, T1 H1102NL, U1 STM32H755IITx, U2 MCP2562FD, U3 SP0504BAHTG, U4 LAN8742A, U5 USBLC6-4SC6, Y1 HS_XTAL, Y2 LS_XTAL

Commit message: more LEDS
Parts:
- removed the C22 at (211.3, 79.6)
- removed the C22 at (173.6, 101.5)
- removed the C23 at (211.3, 82.1)
- removed the C23 at (173.6, 104.0)
- removed IC1: LV14340DDAR, SamacSys_Parts:SOIC127P600X170-9N
- removed IC2: W25M512JVFIQ, SamacSys_Parts:SOIC127P1032X264-16N
- removed L2: 6u, SamacSys_Parts:SRN6028C6R0M
- removed PS1: BU33SD5WG-TR, SamacSys_Parts:SOT95P280X125-5N
- removed PS1: BU33SD5WG-TR, SamacSys_Parts:SOIC127P600X170-9N
- removed T1: H1102NL, SamacSys_Parts:SOIC127P940X597-16N
- added C22: 1u, Capacitor_SMD:C_0603_1608Metric, F.Cu at (128.2, 43.5)
- added C23: 1u, Capacitor_SMD:C_0603_1608Metric, F.Cu at (128.2, 46.0)
- added C28: 5.6p, Capacitor_SMD:C_0603_1608Metric_Pad1.08x0.95mm_HandSolder, F.Cu at (200.1, 89.1)
- added C29: 5.6p, Capacitor_SMD:C_0603_1608Metric_Pad1.08x0.95mm_HandSolder, F.Cu at (208.6, 89.2)
- added C30: 100n, Capacitor_SMD:C_0603_1608Metric_Pad1.08x0.95mm_HandSolder, F.Cu at (82.6, 91.3)
- added C31: 1u, Capacitor_SMD:C_0603_1608Metric_Pad1.08x0.95mm_HandSolder, F.Cu at (82.6, 93.8)
- added C32: 470p, Capacitor_SMD:C_0603_1608Metric_Pad1.08x0.95mm_HandSolder, F.Cu at (82.6, 96.3)
- added C33: 100n, Capacitor_SMD:C_0603_1608Metric_Pad1.08x0.95mm_HandSolder, F.Cu at (82.6, 98.8)
- added C34: 100n, Capacitor_SMD:C_0603_1608Metric_Pad1.08x0.95mm_HandSolder, F.Cu at (82.6, 101.3)
- added C35: 100n, Capacitor_SMD:C_0603_1608Metric_Pad1.08x0.95mm_HandSolder, F.Cu at (82.6, 103.8)
- added C36: 10u, Capacitor_SMD:C_0603_1608Metric_Pad1.08x0.95mm_HandSolder, F.Cu at (82.6, 106.3)
- added C37: 100n, Capacitor_SMD:C_0603_1608Metric_Pad1.08x0.95mm_HandSolder, F.Cu at (82.6, 108.8)
- added C38: 100n, Capacitor_SMD:C_0603_1608Metric_Pad1.08x0.95mm_HandSolder, F.Cu at (87.0, 91.3)
- added C39: 1u, Capacitor_SMD:C_0603_1608Metric_Pad1.08x0.95mm_HandSolder, F.Cu at (87.0, 93.8)
- added D10: LED, LED_SMD:LED_0603_1608Metric, F.Cu at (178.9, 128.1)
- added D11: LED, LED_SMD:LED_0603_1608Metric, F.Cu at (178.9, 130.7)
- added D12: LED, LED_SMD:LED_0603_1608Metric, F.Cu at (178.9, 133.3)
- added D13: LED, LED_SMD:LED_0603_1608Metric, F.Cu at (178.9, 135.9)
- added D14: LED, LED_SMD:LED_0603_1608Metric, F.Cu at (183.0, 125.5)
- added D15: LED, LED_SMD:LED_0603_1608Metric, F.Cu at (183.0, 128.1)
- added D16: LED, LED_SMD:LED_0603_1608Metric, F.Cu at (183.0, 130.7)
- added D2: D, Diode_SMD:D_0603_1608Metric, F.Cu at (174.9, 125.5)
- added D3: D, Diode_SMD:D_0603_1608Metric, F.Cu at (174.9, 128.1)
- added D4: D, Diode_SMD:D_0603_1608Metric, F.Cu at (174.9, 130.7)
- added D5: D, Diode_SMD:D_0603_1608Metric, F.Cu at (174.9, 133.3)
- added D6: PMEG6020AELRX, Diode_SMD:D_SOD-123, F.Cu at (138.8, 102.2)
- added D7: PMEG6020AELRX, Diode_SMD:D_SOD-123, F.Cu at (138.8, 105.6)
- added D8: LED, LED_SMD:LED_0603_1608Metric, F.Cu at (174.9, 135.9)
- added D9: LED, LED_SMD:LED_0603_1608Metric, F.Cu at (178.9, 125.5)
- added J8: USB_B_Micro, Connector_USB:USB_Micro-AB_Molex_47590-0001, F.Cu at (124.3, 115.5)
- added R10: 10K, Resistor_SMD:R_0603_1608Metric, F.Cu at (128.2, 63.5)
- added R11: 1.5K, Resistor_SMD:R_0603_1608Metric, F.Cu at (132.2, 43.5)
- added R12: 10K, Resistor_SMD:R_0603_1608Metric, F.Cu at (132.2, 46.0)
- added R13: 12.1K, Resistor_SMD:R_0603_1608Metric, F.Cu at (132.2, 48.5)
- added R14: 33R, Resistor_SMD:R_0603_1608Metric, F.Cu at (132.2, 51.0)
- added R15: 33R, Resistor_SMD:R_0603_1608Metric, F.Cu at (132.2, 53.5)
- added R16: 33R, Resistor_SMD:R_0603_1608Metric, F.Cu at (132.2, 56.0)
- added R17: 33R, Resistor_SMD:R_0603_1608Metric, F.Cu at (132.2, 58.5)
- added R18: 75R, Resistor_SMD:R_0603_1608Metric, F.Cu at (132.2, 61.0)
- added R19: 75R, Resistor_SMD:R_0603_1608Metric, F.Cu at (132.2, 63.5)
- added R20: 75R, Resistor_SMD:R_0603_1608Metric, F.Cu at (136.2, 43.5)
- added R21: 75R, Resistor_SMD:R_0603_1608Metric, F.Cu at (136.2, 46.0)
- added R22: 10K, Resistor_SMD:R_0603_1608Metric, F.Cu at (136.2, 48.5)
- added R23: 49.9R, Resistor_SMD:R_0603_1608Metric, F.Cu at (136.2, 51.0)
- added R24: 49.9R, Resistor_SMD:R_0603_1608Metric, F.Cu at (136.2, 53.5)
- added R25: 49.9R, Resistor_SMD:R_0603_1608Metric, F.Cu at (136.2, 56.0)
- added R26: 49.9R, Resistor_SMD:R_0603_1608Metric, F.Cu at (136.2, 58.5)
- added R27: 47R, Resistor_SMD:R_0603_1608Metric_Pad0.98x0.95mm_HandSolder, F.Cu at (87.0, 101.3)
- added R28: 330R, Resistor_SMD:R_0603_1608Metric, F.Cu at (215.0, 124.0)
- added R29: 330R, Resistor_SMD:R_0603_1608Metric, F.Cu at (219.5, 124.0)
- added R30: 330R, Resistor_SMD:R_0603_1608Metric, F.Cu at (227.5, 128.0)
- added R31: 330R, Resistor_SMD:R_0603_1608Metric, F.Cu at (223.0, 128.0)
- added R32: 330R, Resistor_SMD:R_0603_1608Metric, F.Cu at (217.5, 128.0)
- added R33: 330R, Resistor_SMD:R_0603_1608Metric, F.Cu at (219.5, 119.5)
- added R34: 330R, Resistor_SMD:R_0603_1608Metric, F.Cu at (227.5, 123.5)
- added R35: 330R, Resistor_SMD:R_0603_1608Metric, F.Cu at (224.0, 124.0)
- added R36: 330R, Resistor_SMD:R_0603_1608Metric, F.Cu at (211.0, 124.0)
- added R7: 10K, Resistor_SMD:R_0603_1608Metric, F.Cu at (128.2, 56.0)
- added R8: 10K, Resistor_SMD:R_0603_1608Metric, F.Cu at (128.2, 58.5)
- added R9: 10K, Resistor_SMD:R_0603_1608Metric, F.Cu at (128.2, 61.0)
- added SB1: NC, Jumper:SolderJumper-2_P1.3mm_Open_TrianglePad1.0x1.5mm, F.Cu at (104.7, 31.9)
- added SB2: NC, Jumper:SolderJumper-2_P1.3mm_Open_TrianglePad1.0x1.5mm, F.Cu at (104.7, 35.5)
- added Y4: HS_XTAL, Crystal:Crystal_SMD_2016-4Pin_2.0x1.6mm, F.Cu at (204.3, 89.5)
- R2: value 10k -> 47R
- moved J2 175.9 mm to (28.8, 49.2), turned to 90 degrees
- moved J3 171.3 mm to (29.0, 74.0), turned to 90 degrees
- moved J9 153.9 mm to (257.0, 69.4), turned to 90 degrees
- moved Y1 124.2 mm to (64.3, 60.0)
- moved C10 121.1 mm to (68.9, 103.0)
- moved C7 121.1 mm to (68.9, 95.5)
- moved C8 121.1 mm to (68.9, 98.0)
- moved C9 121.1 mm to (68.9, 100.5)
- moved U5 116.9 mm to (226.4, 60.0), turned to 180 degrees
- moved R1 101.5 mm to (87.0, 96.3)
- moved R2 101.5 mm to (87.0, 98.8)
- moved U4 90.9 mm to (225.5, 74.2)
- moved Y2 87.3 mm to (72.0, 50.0), turned to 90 degrees
- moved K1 85.1 mm to (40.3, 116.9)
- moved K2 85.1 mm to (49.5, 116.9)
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Connections:
- net /FDCAN_TXD renamed /CAN dataline LED
- net Net-(D2-A) renamed /24V backup LED
- net Net-(D3-A) renamed /24V LED
- C1 pad 1: 3V3 -> +3V3
- C2 pad 1: 3V3 -> +3V3
- C20 pad 1: 5V -> /INT_5V
- C21 pad 1: 5V -> /INT_5V
- C26 pad 1: Net-(U2-VSS) -> GND
- C27 pad 2: 5V -> +5V
- C3 pad 1: 3V3 -> +3V3
- C4 pad 1: 3V3 -> +3V3
- C5 pad 1: 3V3 -> +3V3
- C6 pad 1: 3V3 -> +3V3
- C7 pad 1: 3V3 -> +3V3
- C8 pad 1: GND -> /RESET
- C8 pad 2: 3V3 -> GND
- J9 pad 1: unconnected-(J9-Pad1) -> Net-(T1-TX+)
- J9 pad 2: unconnected-(J9-Pad2) -> Net-(T1-TX-)
- J9 pad 3: unconnected-(J9-Pad3) -> Net-(T1-RX+)
- J9 pad 4: unconnected-(J9-Pad4) -> Net-(T1-RX-)
- J9 pad 5: unconnected-(J9-Pad5) -> Net-(U4-LED1/REGOFF)
- J9 pad 6: unconnected-(J9-Pad6) -> Net-(J9-Pad6)
- J9 pad 8: unconnected-(J9-Pad8) -> Net-(J9-Pad8)
- R1 pad 1: 3V3 -> +3V3
- R2 pad 1: /RESET -> /STL_SWDIO
- R2 pad 2: GND -> /SWDIO
- R3 pad 1: 5V -> /INT_5V
- SW1 pad 1: 3V3 -> GND
- U1 pad 105: 3V3 -> +3V3
- U1 pad 113: 3V3 -> +3V3
- U1 pad 126: 3V3 -> +3V3
- U1 pad 13: 3V3 -> +3V3
- U1 pad 132: unconnected-(U1-PA13-Pad132) -> /SWDIO
- U1 pad 135: 3V3 -> +3V3
- U1 pad 136: 3V3 -> +3V3
- U1 pad 138: unconnected-(U1-PA14-Pad138) -> /SWCLK
- U1 pad 152: 3V3 -> +3V3
- U1 pad 155: unconnected-(U1-PG11-Pad155) -> /ETH_TXEN
- U1 pad 157: unconnected-(U1-PG13-Pad157) -> /ETH_TXD0
- U1 pad 160: 3V3 -> +3V3
- U1 pad 175: 3V3 -> +3V3
- U1 pad 176: 3V3 -> +3V3
- U1 pad 25: 3V3 -> +3V3
- U1 pad 35: unconnected-(U1-PC1-Pad35) -> /ETH_MDC
- U1 pad 39: 3V3 -> +3V3
- U1 pad 40: 3V3 -> +3V3
- U1 pad 42: unconnected-(U1-PA1-Pad42) -> /ETH_REF_CLK
- U1 pad 43: unconnected-(U1-PA2-Pad43) -> /ETH_MDIO
- U1 pad 44: 3V3 -> +3V3
- U1 pad 48: 3V3 -> +3V3
- U1 pad 52: unconnected-(U1-PA7-Pad52) -> /ETH_CRS_DV
- U1 pad 53: unconnected-(U1-PC4-Pad53) -> /ETH_RXD0
- U1 pad 54: unconnected-(U1-PC5-Pad54) -> /ETH_RXD1
- U1 pad 65: 3V3 -> +3V3
- U1 pad 7: 3V3 -> +3V3
- U1 pad 71: 3V3 -> +3V3
- U1 pad 75: /SPI4_MISO -> /FLASH_SPI_MISO
- U1 pad 76: /SPI4_MOSI -> /FLASH_SPI_MOSI
- U1 pad 82: 3V3 -> +3V3
- U1 pad 84: 3V3 -> +3V3
- U1 pad 86: unconnected-(U1-PB13-Pad86) -> /ETH_TXD1
- U1 pad 92: 3V3 -> +3V3
- U1 pad 97: unconnected-(U1-PD14-Pad97) -> /other debug LED
- U1 pad 98: unconnected-(U1-PD15-Pad98) -> /heartbeat LED
- U1 pad 99: 3V3 -> +3V3
- U2 pad 2: Net-(U2-VSS) -> GND
- U2 pad 3: 5V -> +5V
- U4 pad 1: unconnected-(U4-VDD2A-Pad1) -> /ETH pwr LED
- U4 pad 10: unconnected-(U4-RXER/PHYAD0-Pad10) -> Net-(U4-RXER/PHYAD0)
- U4 pad 11: unconnected-(U4-CRS_DV/MODE2-Pad11) -> Net-(U4-CRS_DV/MODE2)
- U4 pad 12: unconnected-(U4-MDIO-Pad12) -> /ETH_MDIO
- U4 pad 13: unconnected-(U4-MDC-Pad13) -> /ETH_MDC
- U4 pad 14: unconnected-(U4-~{INT}/REFCLKO-Pad14) -> Net-(U4-~{INT}/REFCLKO)
- U4 pad 15: unconnected-(U4-~{RST}-Pad15) -> /RESET
- U4 pad 16: unconnected-(U4-TXEN-Pad16) -> /ETH_TXEN
- U4 pad 17: unconnected-(U4-TXD0-Pad17) -> /ETH_TXD0
- U4 pad 18: unconnected-(U4-TXD1-Pad18) -> /ETH_TXD1
- U4 pad 19: unconnected-(U4-VDD1A-Pad19) -> /ETH pwr LED
- U4 pad 2: unconnected-(U4-LED2/~{INTSEL}-Pad2) -> Net-(U4-LED2/~{INTSEL})
- U4 pad 20: unconnected-(U4-TXN-Pad20) -> Net-(T1-TD-)
- U4 pad 21: unconnected-(U4-TXP-Pad21) -> Net-(T1-TD+)
- U4 pad 22: unconnected-(U4-RXN-Pad22) -> Net-(T1-RD-)
- U4 pad 23: unconnected-(U4-RXP-Pad23) -> Net-(T1-RD+)
- U4 pad 24: unconnected-(U4-RBIAS-Pad24) -> Net-(U4-RBIAS)
- U4 pad 25: unconnected-(U4-VSS-Pad25) -> GND
- U4 pad 3: unconnected-(U4-LED1/REGOFF-Pad3) -> Net-(U4-LED1/REGOFF)
- U4 pad 4: unconnected-(U4-XTAL2-Pad4) -> Net-(U4-XTAL2)
- U4 pad 5: unconnected-(U4-XTAL1/CLKIN-Pad5) -> Net-(U4-XTAL1/CLKIN)
- U4 pad 6: unconnected-(U4-VDDCR-Pad6) -> Net-(U4-VDDCR)
- U4 pad 7: unconnected-(U4-RXD1/MODE1-Pad7) -> Net-(U4-RXD1/MODE1)
- U4 pad 8: unconnected-(U4-RXD0/MODE0-Pad8) -> Net-(U4-RXD0/MODE0)
- U4 pad 9: unconnected-(U4-VDDIO-Pad9) -> 3V3
- U5 pad 1: unconnected-(U5-I/O1-Pad1) -> Net-(T1-TD+)
- U5 pad 2: unconnected-(U5-GND-Pad2) -> GND
- U5 pad 3: unconnected-(U5-I/O2-Pad3) -> Net-(T1-TD-)
- U5 pad 4: unconnected-(U5-I/O3-Pad4) -> Net-(T1-RD+)
- U5 pad 5: unconnected-(U5-VBUS-Pad5) -> Net-(U5-VBUS)
- U5 pad 6: unconnected-(U5-I/O4-Pad6) -> Net-(T1-RD-)
Other:
- board outline added: 7.5 x 2 mm
