File: STM32H755_template/STM32H755_template.kicad_sch (KiCad schematic)
At the start: 89 parts, among them IC2 W25M512JVFIQ, J2 melex ultra fit, J3 melex ultra fit, J4 molex ultrafit, J5 molex ultrafit, J6 molex ultrafit, J7 molex ultrafit, J8 USB_B_Micro, J9 RJ45, K1 EC2-3NU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

Commit message: more LEDS
Parts:
- removed SB: NC, Jumper:SolderJumper-2_P1.3mm_Open_TrianglePad1.0x1.5mm, symbol Jumper:SolderJumper_2_Open
- added D10, D11, D12, D13, D14, D15, D16, D8, D9: LED, LED_SMD:LED_0603_1608Metric, symbol Device:LED
- added R28, R29, R30, R31, R32, R33, R34, R35, R36: 330R, Resistor_SMD:R_0603_1608Metric, symbol Device:R
- added SB2: NC, Jumper:SolderJumper-2_P1.3mm_Open_TrianglePad1.0x1.5mm, symbol Jumper:SolderJumper_2_Open
- D2, D3, D4, D5: footprint (none) -> Diode_SMD:D_0603_1608Metric
Connections:
- net +3V3: now also D16.2 (A); no longer C26.2, C30.2, C33.1, L1.2, R10.1, R11.1, R12.1, R8.1, R9.1, U2.5 (Vio), U2.8 (STBY), U4.9 (VDDIO)
- net +5V: now also C27.2, U2.3 (VDD), D12.2 (A)
- net 5V: now also D15.2 (A); no longer C27.2, U2.3 (VDD)
- net FLASH_SPI_MOSI: now also SB2.2 (B)
- net GND: now also C26.1, U2.2 (VSS), R28.2, R29.2, R30.2, R31.2, R32.2, R33.2, R34.2, R35.2, R36.2; no longer C37.1, C38.1, R23.1, R24.1, R25.1, R26.1, T1.2 (CT_1), T1.7 (CT_2)
- net QSPI_IO0: now also SB2.1 (A)
- net ETH pwr LED: now reaches C34.1, C35.1, C36.1, L1.1, U4.1 (VDD2A), U4.19 (VDD1A)
- net ETH pwr LED: now also C37.1, C38.1, R23.1, R24.1, R25.1, R26.1, T1.2 (CT_1), T1.7 (CT_2), D11.2 (A)
- net other debug LED: now reaches U1.97 (PD14)
- net other debug LED: now also D9.2 (A)
- net heartbeat LED: now reaches U1.98 (PD15)
- net heartbeat LED: now also D8.2 (A)
- net 24V LED: now reaches D3.2 (A), J2.5, J3.5
- net 24V LED: now also D14.2 (A)
- net 24V backup LED: now reaches D2.2 (A), J2.6, J3.6
- net 24V backup LED: now also D13.2 (A)
- net FDCAN_TXD renamed CAN dataline LED
- net CAN dataline LED: now also D10.2 (A)
- new net: D10.1 (K), R30.1
- new net: D11.1 (K), R31.1
- new net: D8.1 (K), R28.1
- new net: D13.1 (K), R33.1
- new net: D9.1 (K), R29.1
- new net: D15.1 (K), R35.1
- new net: D12.1 (K), R32.1
- new net: D14.1 (K), R34.1
- new net: D16.1 (K), R36.1
- new net 3V3: C26.2, C30.2, C33.1, L1.2, R10.1, R11.1, R12.1, R8.1, R9.1, U2.5 (Vio), U2.8 (STBY), U4.9 (VDDIO)
- no-connect marks 116 -> 118
Other:
- note added: "change CAN data line LED"
- note added: "debug LED"
- moved on the sheet: C34, C35, C36, L1
